File: meteo_mini.sch (KiCad schematic (older format))
At the start: 15 parts, among them J1 Conn_01x04, J2 Conn_01x06, J3 Conn_01x04, J4 USB_A, SW1 SW_SPST, U1 STM32F103C8T6, U2 XC6206PxxxMR

Commit message: new pcb design is coming
Parts:
- removed J2: Conn_01x06, Connector_PinHeader_2.54mm:PinHeader_1x06_P2.54mm_Vertical, symbol Connector_Generic:Conn_01x06
- added C7: 1u, Capacitor_SMD:C_0603_1608Metric, symbol Device:C
- added C8: 0.1u, Capacitor_SMD:C_0603_1608Metric, symbol Device:C
- added D1, D2: LED, LED_SMD:LED_0603_1608Metric, symbol Device:LED
- added R3, R4: 10k, Resistor_SMD:R_0603_1608Metric, symbol Device:R
- added R5, R6: 390, Resistor_SMD:R_0603_1608Metric, symbol Device:R
- added U3: BME280, Package_LGA:Bosch_LGA-8_2.5x2.5mm_P0.65mm_ClockwisePinNumbering, symbol Sensor:BME280
- C4: footprint Capacitor_SMD:C_0805_2012Metric -> Capacitor_SMD:C_0603_1608Metric
- SW1: footprint Button_Switch_SMD:SW_SPST_REED_CT05-XXXX-J1 -> Button_Switch_SMD:SW_SPST_PTS645
Connections:
- net labels added: LED
- wire segments 76 -> 88
- no-connect marks 36 -> 35
Other:
- note added: "BME280"
- note added: "LED\n"
- moved on the sheet: J1, J3, J4

Commit message: Move components
Parts:
- J1: renamed from J4; symbol Connector:USB_A -> meteo_mini-rescue:USB_A-Connector
- SW1: footprint Button_Switch_SMD:SW_SPST_PTS645 -> Button_Switch_SMD:SW_SPST_FSMSM
- renumbered C7 to C1, C8 to C2, C4 to C3, C5 to C4, C1 to C5, C2 to C6, C6 to C7, C3 to C8, J3 to J2, J1 to J3, R3 to R1, R4 to R2, R5 to R3, R6 to R4, R1 to R5, R2 to R6, U3 to U1, U1 to U2, U2 to U3

Commit message: First version
Parts:
- J1: symbol meteo_mini-rescue:USB_A-Connector -> meteo_mini-rescue:USB_A-Connector-meteo_mini-rescue
Changed lines of the file:
@@
 $EndComp
 $Comp
-L meteo_mini-rescue:USB_A-Connector J1
+L meteo_mini-rescue:USB_A-Connector-meteo_mini-rescue J1
 U 1 1 5F65E491
 P 1450 1645
@@
 Wire Wire Line
 	2325 6325 2325 6225
+Text Notes 1800 5675 0    197  ~ 0
+LED\n
 Text Label 2325 6225 0    50   ~ 0
 LED
-Text Notes 1800 5675 0    197  ~ 0
-LED\n
 $EndSCHEMATC

Commit message: New PCB production
Connections:
- no-connect marks 35 -> 34
Changed lines of the file:
@@
 	-1   0    0    1
 $EndComp
-NoConn ~ 5075 2275
 $Comp
 L power:+5V #PWR018
@@
 Text Label 875  4125 0    50   ~ 0
 I2C1SCL
-$Comp
-L MCU_ST_STM32F1:STM32F103C8Tx U2
-U 1 1 5EBD74CA
-P 5550 2900
-F 0 "U2" H 5500 1311 50  0001 C CNN
-F 1 "STM32F103C8T6" H 5500 1220 50  0001 C CNN
-F 2 "Package_QFP:LQFP-48_7x7mm_P0.5mm" H 4950 1500 50  0001 R CNN
-F 3 "http://www.st.com/st-web-ui/static/active/en/resource/technical/document/datasheet/CD00161566.pdf" H 5550 2900 50  0001 C CNN
-	1    5550 2900
-	1    0    0    -1
-$EndComp
 $Comp
 L power:+3.3V #PWR017
@@
 Text Label 2325 6225 0    50   ~ 0
 LED
+$Comp
+L MCU_ST_STM32F1:STM32F103C8Tx U2
+U 1 1 5EBD74CA
+P 5550 2900
+F 0 "U2" H 5500 1311 50  0001 C CNN
+F 1 "STM32F103C8T6" H 5500 1220 50  0001 C CNN
+F 2 "Package_QFP:LQFP-48_7x7mm_P0.5mm" H 4950 1500 50  0001 R CNN
+F 3 "http://www.st.com/st-web-ui/static/active/en/resource/technical/document/datasheet/CD00161566.pdf" H 5550 2900 50  0001 C CNN
+	1    5550 2900
+	1    0    0    -1
+$EndComp
 $EndSCHEMATC
